Commit message: Update run_simulation to accept inline commands

File: bocbot_ws/src/bocbot/urdf/bocbot.urdf (robot description, URDF)
Before this commit: robot bocbot, 8 links, 7 joints
Links:
- removed link chassis
- added link base_link, mass 15.0; collision box size=0.35 0.25 0.15; visual box size=0.35 0.25 0.15
- added link left_bogie_link, mass 1.5; collision box size=0.25 0.04 0.04; visual box size=0.25 0.04 0.04
- added link left_rocker_arm, mass 2.0; collision box size=0.3 0.05 0.05; visual box size=0.3 0.05 0.05
- added link mid_left_wheel, mass 2.0; collision cylinder length=0.06 radius=0.075; visual cylinder length=0.06 radius=0.075
- added link mid_right_wheel, mass 2.0; collision cylinder length=0.06 radius=0.075; visual cylinder length=0.06 radius=0.075
- added link right_bogie_link, mass 1.5; collision box size=0.25 0.04 0.04; visual box size=0.25 0.04 0.04
- added link right_rocker_arm, mass 2.0; collision box size=0.3 0.05 0.05; visual box size=0.3 0.05 0.05
- link back_left_wheel: mass 5.0 -> 2.0; geometry collision cylinder length=0.06 radius=0.075; visual cylinder length=0.06 radius=0.075
- link back_right_wheel: mass 5.0 -> 2.0; geometry collision cylinder length=0.06 radius=0.075; visual cylinder length=0.06 radius=0.075
- link front_left_wheel: mass 5.0 -> 2.0; geometry collision cylinder length=0.06 radius=0.075; visual cylinder length=0.06 radius=0.075
- link front_right_wheel: mass 5.0 -> 2.0; geometry collision cylinder length=0.06 radius=0.075; visual cylinder length=0.06 radius=0.075
Joints:
- added joint left_bogie_pivot: type revolute, parent left_rocker_arm, child left_bogie_link, origin xyz=-0.2 0.0 0 rpy=0 0 0, axis 0 1 0, limit lower=-0.78 upper=0.78 effort=500 velocity=100
- added joint left_differential_axle: type revolute, parent base_link, child left_rocker_arm, origin xyz=0.0 0.15 0 rpy=0 0 0, axis 0 1 0, limit lower=-0.78 upper=0.78 effort=1000 velocity=100
- added joint mid_left_wheel_joint: type continuous, parent left_bogie_link, child mid_left_wheel, origin xyz=0.0 0.05 -0.1 rpy=0 0 0, axis 0 1 0, limit effort=10000 velocity=1000
- added joint mid_right_wheel_joint: type continuous, parent right_bogie_link, child mid_right_wheel, origin xyz=0.0 -0.05 -0.1 rpy=0 0 0, axis 0 1 0, limit effort=10000 velocity=1000
- added joint right_bogie_pivot: type revolute, parent right_rocker_arm, child right_bogie_link, origin xyz=-0.2 0.0 0 rpy=0 0 0, axis 0 1 0, limit lower=-0.78 upper=0.78 effort=500 velocity=100
- added joint right_differential_axle: type revolute, parent base_link, child right_rocker_arm, origin xyz=0.0 -0.15 0 rpy=0 0 0, axis 0 1 0, limit lower=-0.78 upper=0.78 effort=1000 velocity=100
- joint back_left_wheel_joint: origin xyz=-0.12 0.15 0 rpy=0 0 0 -> xyz=-0.2 0.05 -0.1 rpy=0 0 0; parent chassis -> left_bogie_link
- joint back_right_wheel_joint: origin xyz=-0.12 -0.15 0 rpy=0 0 0 -> xyz=-0.2 -0.05 -0.1 rpy=0 0 0; parent chassis -> right_bogie_link
- joint camera_joint: origin xyz=0.2 0 0 rpy=0 0 0 -> xyz=0.175 0 0 rpy=0 0 0; parent chassis -> base_link
- joint front_left_wheel_joint: origin xyz=0.12 0.15 0 rpy=0 0 0 -> xyz=0.1 0.05 -0.1 rpy=0 0 0; parent chassis -> left_rocker_arm
- joint front_right_wheel_joint: origin xyz=0.12 -0.15 0 rpy=0 0 0 -> xyz=0.1 -0.05 -0.1 rpy=0 0 0; parent chassis -> right_rocker_arm
- joint hokuyo_joint: origin xyz=0.15 0 0.1 rpy=0 0 0 -> xyz=0 0 0.1 rpy=0 0 0; parent chassis -> base_link
- joint robot_footprint_joint: child chassis -> base_link

File: bocbot_ws/src/bocbot/urdf/bocbot.urdf.xacro (robot description, xacro)
@@ -1,17 +1,18 @@
 <?xml version='1.0'?>
-<robot name="bocbot"
-  xmlns:xacro="http://www.ros.org/wiki/xacro">
+<robot name="bocbot" xmlns:xacro="http://www.ros.org/wiki/xacro">
   <xacro:include filename="bocbot.gazebo" />
+  <!-- Base footprint -->
   <link name="robot_footprint"></link>
   <joint name="robot_footprint_joint" type="fixed">
     <origin xyz="0 0 0" rpy="0 0 0" />
     <parent link="robot_footprint"/>
-    <child link="chassis" />
-  </joint>
-  <link name='chassis'>
-    <pose>0 0 0.1 0 0 0</pose>
+    <child link="base_link" />
+  </joint>
+  <!-- Main Chassis (Green/White Box from images) -->
+  <link name='base_link'>
+    <pose>0 0 0.2 0 0 0</pose>
     <inertial>
       <mass value="15.0"/>
-      <origin xyz="0.0 0 0" rpy=" 0 0 0"/>
+      <origin xyz="0 0 0" rpy=" 0 0 0"/>
       <inertia ixx="0.1" ixy="0" ixz="0" iyy="0.1" iyz="0" izz="0.1" />
     </inertial>
@@ -19,5 +20,6 @@
       <origin xyz="0 0 0" rpy=" 0 0 0"/>
       <geometry>
-        <box size=".4 .2 .1"/>
+        <!-- Polyhedral shape approximated as a box for now -->
+        <box size="0.35 0.25 0.15"/>
       </geometry>
     </collision>
@@ -25,88 +27,17 @@
       <origin xyz="0 0 0" rpy=" 0 0 0"/>
       <geometry>
-        <box size=".4 .2 .1"/>
-      </geometry>
-    </visual>
-  </link>
-  <link name="front_left_wheel">
-    <inertial>
-      <mass value="5.0"/>
-      <origin xyz="0.0 0 0" rpy=" 0 1.5707 1.5707"/>
-      <inertia ixx="0.1" ixy="0" ixz="0" iyy="0.1" iyz="0" izz="0.1" />
-    </inertial>
-    <visual>
-      <origin xyz="0.0 0 0" rpy=" 0 1.5707 1.5707"/>
-      <geometry>
-        <cylinder length="0.05" radius="0.1"/>
-      </geometry>
-    </visual>
-    <collision>
-      <origin xyz="0.0 0 0" rpy=" 0 1.5707 1.5707"/>
-      <geometry>
-        <cylinder length="0.05" radius="0.1"/>
-      </geometry>
-    </collision>
-  </link>
-  <link name="back_left_wheel">
-    <inertial>
-      <mass value="5.0"/>
-      <origin xyz="0.0 0 0" rpy=" 0 1.5707 1.5707"/>
-      <inertia ixx="0.1" ixy="0" ixz="0" iyy="0.1" iyz="0" izz="0.1" />
-    </inertial>
-    <visual>
-      <origin xyz="0.0 0 0" rpy=" 0 1.5707 1.5707"/>
-      <geometry>
-        <cylinder length="0.05" radius="0.1"/>
-      </geometry>
-    </visual>
-    <collision>
-      <origin xyz="0.0 0 0" rpy=" 0 1.5707 1.5707"/>
-      <geometry>
-        <cylinder length="0.05" radius="0.1"/>
-      </geometry>
-    </collision>
-  </link>
-  <link name="front_right_wheel">
-    <inertial>
-      <mass value="5.0"/>
-      <origin xyz="0.0 0 0" rpy=" 0 1.5707 1.5707"/>
-      <inertia ixx="0.1" ixy="0" ixz="0" iyy="0.1" iyz="0" izz="0.1" />
-    </inertial>
-    <visual>
-      <origin xyz="0.0 0 0" rpy=" 0 1.5707 1.5707"/>
-      <geometry>
-        <cylinder length="0.05" radius="0.1"/>
-      </geometry>
-    </visual>
-    <collision>
-      <origin xyz="0.0 0 0" rpy=" 0 1.5707 1.5707"/>
-      <geometry>
-        <cylinder length="0.05" radius="0.1"/>
-      </geometry>
-    </collision>
-  </link>
-  <link name="back_right_wheel">
-    <inertial>
-      <mass value="5.0"/>
-      <origin xyz="0.0 0 0" rpy=" 0 1.5707 1.5707"/>
-      <inertia ixx="0.1" ixy="0" ixz="0" iyy="0.1" iyz="0" izz="0.1" />
-    </inertial>
-    <visual>
-      <origin xyz="0.0 0 0" rpy=" 0 1.5707 1.5707"/>
-      <geometry>
-        <cylinder length="0.05" radius="0.1"/>
-      </geometry>
-    </visual>
-    <collision>
-      <origin xyz="0.0 0 0" rpy=" 0 1.5707 1.5707"/>
-      <geometry>
-        <cylinder length="0.05" radius="0.1"/>
-      </geometry>
-    </collision>
-  </link>
+        <box size="0.35 0.25 0.15"/>
+      </geometry>
+    </visual>
+  </link>
+  <gazebo reference="base_link">
+    <!-- Using Green to match the first two images -->
+    <material>Gazebo/Green</material>
+  </gazebo>
+  <!-- Sensors attached to base_link -->
   <link name="camera">
     <inertial>
       <mass value="0.1"/>
-      <origin xyz="0.05 0.05 0.05" rpy=" 0 0 0"/>
+      <origin xyz="0.0 0.0 0.0" rpy=" 0 0 0"/>
       <inertia ixx="1e-6" ixy="0" ixz="0" iyy="1e-6" iyz="0" izz="1e-6" />
     </inertial>
@@ -133,5 +64,4 @@
       <origin xyz="0 0 0" rpy="0 0 0" />
       <geometry>
-        <!-- <mesh filename="$(find bocbot)/meshes/hokuyo.dae"/> -->
         <box size="0.05 0.05 0.05"/>
       </geometry>
@@ -144,51 +74,18 @@
     </collision>
   </link>
-  <joint type="continuous" name="front_left_wheel_joint">
-    <origin xyz="0.12 0.15 0" rpy="0 0 0"/>
-    <child link="front_left_wheel"/>
-    <parent link="chassis"/>
+  <joint type="fixed" name="camera_joint">
+    <!-- Centered in the front of the green hull -->
+    <origin xyz="0.175 0 0" rpy="0 0 0"/>
+    <child link="camera"/>
+    <parent link="base_link"/>
     <axis xyz="0 1 0" rpy="0 0 0"/>
-    <limit effort="10000" velocity="1000"/>
-    <dynamics damping="1.0" friction="1.0"/>
-  </joint>
-  <joint type="continuous" name="front_right_wheel_joint">
-    <origin xyz="0.12 -0.15 0" rpy="0 0 0"/>
-    <child link="front_right_wheel"/>
-    <parent link="chassis"/>
+  </joint>
+  <joint type="fixed" name="hokuyo_joint">
+    <!-- Mounted on top of the green hull -->
+    <origin xyz="0 0 0.1" rpy="0 0 0"/>
+    <child link="hokuyo"/>
+    <parent link="base_link"/>
     <axis xyz="0 1 0" rpy="0 0 0"/>
-    <limit effort="10000" velocity="1000"/>
-    <dynamics damping="1.0" friction="1.0"/>
-  </joint>
-  <joint type="continuous" name="back_left_wheel_joint">
-    <origin xyz="-0.12 0.15 0" rpy="0 0 0"/>
-    <child link="back_left_wheel"/>
-    <parent link="chassis"/>
-    <axis xyz="0 1 0" rpy="0 0 0"/>
-    <limit effort="10000" velocity="1000"/>
-    <dynamics damping="1.0" friction="1.0"/>
-  </joint>
-  <joint type="continuous" name="back_right_wheel_joint">
-    <origin xyz="-0.12 -0.15 0" rpy="0 0 0"/>
-    <child link="back_right_wheel"/>
-    <parent link="chassis"/>
-    <axis xyz="0 1 0" rpy="0 0 0"/>
-    <limit effort="10000" velocity="1000"/>
-    <dynamics damping="1.0" friction="1.0"/>
-  </joint>
-  <joint type="fixed" name="camera_joint">
-    <origin xyz="0.2 0 0" rpy="0 0 0"/>
-    <child link="camera"/>
-    <parent link="chassis"/>
-    <axis xyz="0 1 0" rpy="0 0 0"/>
-  </joint>
-  <joint type="fixed" name="hokuyo_joint">
-    <origin xyz="0.15 0 0.1" rpy="0 0 0"/>
-    <child link="hokuyo"/>
-    <parent link="chassis"/>
-    <axis xyz="0 1 0" rpy="0 0 0"/>
-  </joint>
-  <gazebo reference="chassis">
-    <material>Gazebo/Blue</material>
-  </gazebo>
+  </joint>
   <gazebo reference="camera">
     <material>Gazebo/Red</material>
@@ -197,3 +94,371 @@
     <material>Gazebo/Black</material>
   </gazebo>
+  <!-- =============================== -->
+  <!-- LEFT SIDE ROCKER-BOGIE ASSEMBLY -->
+  <!-- =============================== -->
+  <!-- Left Main Rocker Arm -->
+  <link name="left_rocker_arm">
+    <inertial>
+      <mass value="2.0"/>
+      <origin xyz="0 0 0" rpy="0 0 0"/>
+      <inertia ixx="0.05" ixy="0" ixz="0" iyy="0.05" iyz="0" izz="0.05" />
+    </inertial>
+    <visual>
+      <origin xyz="-0.05 0.05 -0.05" rpy="0 0 0"/>
+      <geometry>
+        <box size="0.3 0.05 0.05"/>
+      </geometry>
+    </visual>
+    <collision>
+      <origin xyz="-0.05 0.05 -0.05" rpy="0 0 0"/>
+      <geometry>
+        <box size="0.3 0.05 0.05"/>
+      </geometry>
+    </collision>
+  </link>
+  <gazebo reference="left_rocker_arm">
+    <material>Gazebo/DarkGrey</material>
+  </gazebo>
+  <!-- Left Rocker to Chassis Joint (Pitch Revolute) -->
+  <joint name="left_differential_axle" type="revolute">
+    <origin xyz="0.0 0.15 0" rpy="0 0 0"/>
+    <parent link="base_link"/>
+    <child link="left_rocker_arm"/>
+    <axis xyz="0 1 0"/>
+    <limit lower="-0.78" upper="0.78" effort="1000" velocity="100"/>
+    <dynamics damping="5.0" friction="5.0"/>
+  </joint>
+  <!-- Left Front Wheel Module -->
+  <link name="front_left_wheel">
+    <inertial>
+      <mass value="2.0"/>
+      <origin xyz="0 0 0" rpy="1.5707 0 0"/>
+      <inertia ixx="0.01" ixy="0" ixz="0" iyy="0.01" iyz="0" izz="0.01" />
+    </inertial>
+    <visual>
+      <origin xyz="0 0 0" rpy="1.5707 0 0"/>
+      <geometry>
+        <cylinder length="0.06" radius="0.075"/>
+      </geometry>
+    </visual>
+    <collision>
+      <origin xyz="0 0 0" rpy="1.5707 0 0"/>
+      <geometry>
+        <cylinder length="0.06" radius="0.075"/>
+      </geometry>
+      <surface>
+        <friction>
+          <ode>
+            <mu>1.0</mu>
+            <mu2>1.0</mu2>
+          </ode>
+        </friction>
+      </surface>
+    </collision>
+  </link>
+  <gazebo reference="front_left_wheel">
+    <material>Gazebo/Grey</material>
+  </gazebo>
+  <joint name="front_left_wheel_joint" type="continuous">
+    <origin xyz="0.1 0.05 -0.1" rpy="0 0 0"/>
+    <parent link="left_rocker_arm"/>
+    <child link="front_left_wheel"/>
+    <axis xyz="0 1 0"/>
+    <limit effort="10000" velocity="1000"/>
+    <dynamics damping="1.0" friction="1.0"/>
+  </joint>
+  <!-- Left Bogie Link (Trailing) -->
+  <link name="left_bogie_link">
+    <inertial>
+      <mass value="1.5"/>
+      <origin xyz="-0.1 0.05 -0.05" rpy="0 0 0"/>
+      <inertia ixx="0.03" ixy="0" ixz="0" iyy="0.03" iyz="0" izz="0.03" />
+    </inertial>
+    <visual>
+      <origin xyz="-0.1 0.05 -0.05" rpy="0 0 0"/>
+      <geometry>
+        <box size="0.25 0.04 0.04"/>
+      </geometry>
+    </visual>
+    <collision>
+      <origin xyz="-0.1 0.05 -0.05" rpy="0 0 0"/>
+      <geometry>
+        <box size="0.25 0.04 0.04"/>
+      </geometry>
+    </collision>
+  </link>
+  <gazebo reference="left_bogie_link">
+    <material>Gazebo/DarkGrey</material>
+  </gazebo>
+  <!-- Left Rocker to Bogie Joint (Passive Pitch) -->
+  <joint name="left_bogie_pivot" type="revolute">
+    <origin xyz="-0.2 0.0 0" rpy="0 0 0"/>
+    <parent link="left_rocker_arm"/>
+    <child link="left_bogie_link"/>
+    <axis xyz="0 1 0"/>
+    <limit lower="-0.78" upper="0.78" effort="500" velocity="100"/>
+    <dynamics damping="2.0" friction="2.0"/>
+  </joint>
+  <!-- Left Middle Wheel Module -->
+  <link name="mid_left_wheel">
+    <inertial>
+      <mass value="2.0"/>
+      <origin xyz="0 0 0" rpy="1.5707 0 0"/>
+      <inertia ixx="0.01" ixy="0" ixz="0" iyy="0.01" iyz="0" izz="0.01" />
+    </inertial>
+    <visual>
+      <origin xyz="0 0 0" rpy="1.5707 0 0"/>
+      <geometry>
+        <cylinder length="0.06" radius="0.075"/>
+      </geometry>
+    </visual>
+    <collision>
+      <origin xyz="0 0 0" rpy="1.5707 0 0"/>
+      <geometry>
+        <cylinder length="0.06" radius="0.075"/>
+      </geometry>
+      <surface>
+        <friction>
+          <ode>
+            <mu>1.0</mu>
+            <mu2>1.0</mu2>
+          </ode>
+        </friction>
+      </surface>
+    </collision>
+  </link>
+  <gazebo reference="mid_left_wheel">
+    <material>Gazebo/Grey</material>
+  </gazebo>
+  <joint name="mid_left_wheel_joint" type="continuous">
+    <origin xyz="0.0 0.05 -0.1" rpy="0 0 0"/>
+    <parent link="left_bogie_link"/>
+    <child link="mid_left_wheel"/>
+    <axis xyz="0 1 0"/>
+    <limit effort="10000" velocity="1000"/>
+    <dynamics damping="1.0" friction="1.0"/>
+  </joint>
+  <!-- Left Rear Wheel Module -->
+  <link name="back_left_wheel">
+    <inertial>
+      <mass value="2.0"/>
+      <origin xyz="0 0 0" rpy="1.5707 0 0"/>
+      <inertia ixx="0.01" ixy="0" ixz="0" iyy="0.01" iyz="0" izz="0.01" />
+    </inertial>
+    <visual>
+      <origin xyz="0 0 0" rpy="1.5707 0 0"/>
+      <geometry>
+        <cylinder length="0.06" radius="0.075"/>
+      </geometry>
+    </visual>
+    <collision>
+      <origin xyz="0 0 0" rpy="1.5707 0 0"/>
+      <geometry>
+        <cylinder length="0.06" radius="0.075"/>
+      </geometry>
+      <surface>
+        <friction>
+          <ode>
+            <mu>1.0</mu>
+            <mu2>1.0</mu2>
+          </ode>
+        </friction>
+      </surface>
+    </collision>
+  </link>
+  <gazebo reference="back_left_wheel">
+    <material>Gazebo/Grey</material>
+  </gazebo>
+  <joint name="back_left_wheel_joint" type="continuous">
+    <origin xyz="-0.2 0.05 -0.1" rpy="0 0 0"/>
+    <parent link="left_bogie_link"/>
+    <child link="back_left_wheel"/>
+    <axis xyz="0 1 0"/>
+    <limit effort="10000" velocity="1000"/>
+    <dynamics damping="1.0" friction="1.0"/>
+  </joint>
+  <!-- ================================ -->
+  <!-- RIGHT SIDE ROCKER-BOGIE ASSEMBLY -->
+  <!-- ================================ -->
+  <!-- Right Main Rocker Arm -->
+  <link name="right_rocker_arm">
+    <inertial>
+      <mass value="2.0"/>
+      <origin xyz="0 0 0" rpy="0 0 0"/>
+      <inertia ixx="0.05" ixy="0" ixz="0" iyy="0.05" iyz="0" izz="0.05" />
+    </inertial>
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