Commit message: Fix normalized joint axes, simplify ROS topics to global /cmd_vel, and boost monster truck torque

File: bocbot_ws/src/bocbot/urdf/bocbot.urdf (robot description, URDF)
Before this commit: robot bocbot, 15 links, 14 joints
Links:
- link back_left_wheel: mass 0.8 -> 5.0; geometry collision cylinder length=0.2 radius=0.375; visual cylinder length=0.2 radius=0.375
- link back_right_wheel: mass 0.8 -> 5.0; geometry collision cylinder length=0.2 radius=0.375; visual cylinder length=0.2 radius=0.375
- link base_link: mass 4.0 -> 50.0; geometry collision box size=1.2 0.8 0.4; visual box size=1.5 1.0 0.6
- link camera: geometry visual box size=0.1 0.2 0.1
- link front_left_wheel: mass 0.8 -> 5.0; geometry collision cylinder length=0.2 radius=0.375; visual cylinder length=0.2 radius=0.375
- link front_right_wheel: mass 0.8 -> 5.0; geometry collision cylinder length=0.2 radius=0.375; visual cylinder length=0.2 radius=0.375
- link hokuyo: geometry visual cylinder length=0.15 radius=0.1
- link imu_link: mass 0.001 -> 0.01
- link left_bogie_link: mass 0.5 -> 4.0; geometry visual box size=1.2 0.2 0.2
- link left_rocker_arm: mass 0.5 -> 5.0; geometry visual box size=1.7 0.2 0.2
- link mid_left_wheel: mass 0.8 -> 5.0; geometry collision cylinder length=0.2 radius=0.375; visual cylinder length=0.2 radius=0.375
- link mid_right_wheel: mass 0.8 -> 5.0; geometry collision cylinder length=0.2 radius=0.375; visual cylinder length=0.2 radius=0.375
- link right_bogie_link: mass 0.5 -> 4.0; geometry visual box size=1.2 0.2 0.2
- link right_rocker_arm: mass 0.5 -> 5.0; geometry visual box size=1.7 0.2 0.2
Joints:
- joint back_left_wheel_joint: axis 0.0 3.0 0.0 -> 0 1 0; limit effort=100 velocity=20 -> (none); origin xyz=-0.9 0.54 -0.45 rpy=0 0 0 -> xyz=-0.5 0.2 -0.3 rpy=0 0 0
- joint back_right_wheel_joint: axis 0.0 3.0 0.0 -> 0 1 0; limit effort=100 velocity=20 -> (none); origin xyz=-0.9 -0.54 -0.45 rpy=0 0 0 -> xyz=-0.5 -0.2 -0.3 rpy=0 0 0
- joint camera_joint: origin xyz=0.45 0.0 0.0 rpy=0 0 0 -> xyz=0.75 0 0
- joint front_left_wheel_joint: axis 0.0 3.0 0.0 -> 0 1 0; limit effort=100 velocity=20 -> (none); origin xyz=1.8 0.54 -0.9 rpy=0 0 0 -> xyz=1.0 0.2 -0.5 rpy=0 0 0
- joint front_right_wheel_joint: axis 0.0 3.0 0.0 -> 0 1 0; limit effort=100 velocity=20 -> (none); origin xyz=1.8 -0.54 -0.9 rpy=0 0 0 -> xyz=1.0 -0.2 -0.5 rpy=0 0 0
- joint hokuyo_joint: origin xyz=0.3 0.0 0.18 rpy=0 0 0 -> xyz=0.5 0 0.35
- joint imu_joint: origin xyz=0.0 0.0 0.0 rpy=0 0 0 -> xyz=0 0 0
- joint left_bogie_pivot: axis 0.0 3.0 0.0 -> 0 1 0; limit lower=-0.8 upper=0.8 effort=500 velocity=10 -> lower=-0.8 upper=0.8 effort=5000 velocity=5; origin xyz=-0.3 0.0 -0.15 rpy=0 0 0 -> xyz=-0.5 0 -0.2 rpy=0 0 0
- joint left_differential_axle: axis 0.0 3.0 0.0 -> 0 1 0; limit lower=-0.6 upper=0.6 effort=1000 velocity=10 -> lower=-0.6 upper=0.6 effort=10000 velocity=5; origin xyz=0.0 0.39 0.0 rpy=0 0 0 -> xyz=0.0 0.65 0 rpy=0 0 0
- joint mid_left_wheel_joint: axis 0.0 3.0 0.0 -> 0 1 0; limit effort=100 velocity=20 -> (none); origin xyz=0.9 0.54 -0.45 rpy=0 0 0 -> xyz=0.5 0.2 -0.3 rpy=0 0 0
- joint mid_right_wheel_joint: axis 0.0 3.0 0.0 -> 0 1 0; limit effort=100 velocity=20 -> (none); origin xyz=0.9 -0.54 -0.45 rpy=0 0 0 -> xyz=0.5 -0.2 -0.3 rpy=0 0 0
- joint right_bogie_pivot: axis 0.0 3.0 0.0 -> 0 1 0; limit lower=-0.8 upper=0.8 effort=500 velocity=10 -> lower=-0.8 upper=0.8 effort=5000 velocity=5; origin xyz=-0.3 0.0 -0.15 rpy=0 0 0 -> xyz=-0.5 0 -0.2 rpy=0 0 0
- joint right_differential_axle: axis 0.0 3.0 0.0 -> 0 1 0; limit lower=-0.6 upper=0.6 effort=1000 velocity=10 -> lower=-0.6 upper=0.6 effort=10000 velocity=5; origin xyz=0.0 -0.39 0.0 rpy=0 0 0 -> xyz=0.0 -0.65 0 rpy=0 0 0
- joint robot_footprint_joint: origin xyz=0.0 0.0 0.45 rpy=0 0 0 -> xyz=0 0 1.5 rpy=0 0 0

File: bocbot_ws/src/bocbot/urdf/bocbot.urdf.xacro (robot description, xacro)
@@ -2,105 +2,74 @@
 <robot name="bocbot" xmlns:xacro="http://www.ros.org/wiki/xacro">
   <xacro:include filename="bocbot.gazebo" />
-  <!-- ======================================================== -->
-  <!-- ROBOTIC MECHANICS & KINEMATICS UPGRADE                   -->
-  <!-- ======================================================== -->
   <link name="robot_footprint"></link>
   <joint name="robot_footprint_joint" type="fixed">
-    <origin xyz="0.0 0.0 0.45" rpy="0 0 0" />
+    <!-- GIANT SCALE SPAWN: 1.5m in the air to allow the monster wheels to unfold -->
+    <origin xyz="0 0 1.5" rpy="0 0 0" />
     <parent link="robot_footprint"/>
     <child link="base_link" />
   </joint>
-  <!-- Main Chassis -->
+  <!-- ======================================================== -->
+  <!-- MAIN CHASSIS - 5X SCALE (1.5m Length)                    -->
+  <!-- ======================================================== -->
   <link name='base_link'>
     <inertial>
-      <mass value="4.0"/>
-      <!-- ADVANCED MECHANICS: Lowering the Center of Mass (CoM).
-           By shifting the Z origin of the inertia down by 5cm (-0.05),
-           we simulate a heavy battery pack mounted at the very bottom
-           of the hull. This mathematically increases the tip-over angle,
-           making it exceptionally stable on steep stairs. -->
-      <origin xyz="0.0 0.0 -0.15" rpy=" 0 0 0"/>
-      <inertia ixx="0.05" ixy="0" ixz="0" iyy="0.05" iyz="0" izz="0.05" />
+      <mass value="50.0"/>
+      <!-- Heavy underbelly battery simulation -->
+      <origin xyz="0 0 -0.2" rpy=" 0 0 0"/>
+      <inertia ixx="5.0" ixy="0" ixz="0" iyy="8.0" iyz="0" izz="10.0" />
     </inertial>
     <collision name='collision'>
-      <origin xyz="0.0 0.0 0.0" rpy=" 0 0 0"/>
-      <geometry><box size="0.84 0.54 0.3"/></geometry>
+      <origin xyz="0 0 0" rpy=" 0 0 0"/>
+      <geometry><box size="1.2 0.8 0.4"/></geometry>
     </collision>
     <visual name='chassis_visual'>
-      <origin xyz="0.0 0.0 0.0" rpy=" 0 0 0"/>
-      <geometry><box size="0.9 0.6 0.36"/></geometry>
+      <origin xyz="0 0 0" rpy=" 0 0 0"/>
+      <geometry><box size="1.5 1.0 0.6"/></geometry>
     </visual>
   </link>
   <gazebo reference="base_link"><material>Gazebo/Green</material></gazebo>
-  <!-- IMU Sensor Link (New System Component) -->
-  <link name="imu_link">
-    <inertial>
-      <mass value="0.001"/>
-      <origin xyz="0.0 0.0 0.0" rpy="0 0 0"/>
-      <inertia ixx="1e-6" ixy="0" ixz="0" iyy="1e-6" iyz="0" izz="1e-6" />
-    </inertial>
-  </link>
-  <joint name="imu_joint" type="fixed">
-    <origin xyz="0.0 0.0 0.0" rpy="0 0 0" />
-    <parent link="base_link"/>
-    <child link="imu_link" />
-  </joint>
-  <!-- Camera -->
+  <link name="imu_link"><inertial><mass value="0.01"/><origin xyz="0 0 0"/><inertia ixx="1e-6" ixy="0" ixz="0" iyy="1e-6" iyz="0" izz="1e-6"/></inertial></link>
+  <joint name="imu_joint" type="fixed"><origin xyz="0 0 0"/><parent link="base_link"/><child link="imu_link"/></joint>
   <link name="camera">
-    <visual name="camera_visual">
-      <origin xyz="0.0 0.0 0.0" rpy="0 0 0" />
-      <geometry><box size="0.09 0.15 0.09"/></geometry>
-    </visual>
+    <visual><origin xyz="0 0 0"/><geometry><box size="0.1 0.2 0.1"/></geometry></visual>
   </link>
   <joint type="fixed" name="camera_joint">
-    <origin xyz="0.45 0.0 0.0" rpy="0 0 0"/>
-    <child link="camera"/>
-    <parent link="base_link"/>
+    <origin xyz="0.75 0 0"/><child link="camera"/><parent link="base_link"/>
   </joint>
   <gazebo reference="camera"><material>Gazebo/Black</material></gazebo>
-  <!-- Hokuyo LiDAR -->
   <link name="hokuyo">
-    <visual name="hokuyo_visual">
-      <origin xyz="0.0 0.0 0.0" rpy="0 0 0" />
-      <geometry><cylinder radius="0.03" length="0.04"/></geometry>
-    </visual>
+    <visual><origin xyz="0 0 0"/><geometry><cylinder radius="0.1" length="0.15"/></geometry></visual>
   </link>
   <joint type="fixed" name="hokuyo_joint">
-    <origin xyz="0.3 0.0 0.18" rpy="0 0 0"/>
-    <child link="hokuyo"/>
-    <parent link="base_link"/>
+    <origin xyz="0.5 0 0.35"/><child link="hokuyo"/><parent link="base_link"/>
   </joint>
   <gazebo reference="hokuyo"><material>Gazebo/Black</material></gazebo>
   <!-- ======================================================== -->
-  <!-- MACROS FOR CLEAN CODE (Professional Robotics Standard)   -->
+  <!-- MONSTER WHEEL MACRO                                      -->
   <!-- ======================================================== -->
   <xacro:macro name="boc_wheel" params="name parent origin_xyz">
     <link name="${name}">
       <inertial>
-        <mass value="0.8"/>
-        <origin xyz="0.0 0.0 0.0" rpy="1.5707 0 0"/>
-        <inertia ixx="0.0013" ixy="0" ixz="0" iyy="0.0013" iyz="0" izz="0.0022" />
+        <mass value="5.0"/>
+        <origin xyz="0 0 0" rpy="1.570796 0 0"/>
+        <!-- Proportional inertia for large cylinder -->
+        <inertia ixx="0.2" ixy="0" ixz="0" iyy="0.2" iyz="0" izz="0.35" />
       </inertial>
       <visual>
-        <origin xyz="0.0 0.0 0.0" rpy="1.5707 0 0"/>
-        <geometry><cylinder length="0.05" radius="0.075"/></geometry>
+        <origin xyz="0 0 0" rpy="1.570796 0 0"/>
+        <geometry><cylinder length="0.2" radius="0.375"/></geometry>
       </visual>
       <collision>
-        <origin xyz="0.0 0.0 0.0" rpy="1.5707 0 0"/>
-        <geometry><cylinder length="0.05" radius="0.075"/></geometry>
+        <origin xyz="0 0 0" rpy="1.570796 0 0"/>
+        <geometry><cylinder length="0.2" radius="0.375"/></geometry>
       </collision>
     </link>
     <gazebo reference="${name}">
       <material>Gazebo/Grey</material>
-      <!-- ADVANCED MECHANICS: Anisotropic Friction.
-           In a 6-wheel skid steer, the wheels MUST slip sideways to turn.
-           mu1 (forward friction) is high (1.2) for stair climbing grip.
-           mu2 (lateral friction) is extremely low (0.1) so the robot
-           can easily rotate on its center axis without fighting itself! -->
-      <mu1>1.2</mu1>
-      <mu2>0.1</mu2>
+      <!-- Optimized for massive rover turning -->
+      <mu1>1.5</mu1>
+      <mu2>0.02</mu2> <!-- Almost zero lateral friction to allow easy pivot -->
       <kp>1000000.0</kp>
       <kd>100.0</kd>
-      <minDepth>0.001</minDepth>
     </gazebo>
     <joint name="${name}_joint" type="continuous">
@@ -108,7 +77,6 @@
       <parent link="${parent}"/>
       <child link="${name}"/>
-      <axis xyz="0.0 3.0 0.0"/>
-      <limit effort="100" velocity="20"/>
-      <dynamics damping="0.1" friction="0.1"/>
+      <axis xyz="0 1 0"/>
+      <dynamics damping="0.5" friction="0.5"/>
     </joint>
   </xacro:macro>
@@ -118,52 +86,40 @@
   <link name="left_rocker_arm">
     <inertial>
-      <mass value="0.5"/>
-      <origin xyz="0.15 0.0 0.0" rpy="0 0 0"/>
-      <inertia ixx="0.005" ixy="0" ixz="0" iyy="0.005" iyz="0" izz="0.005" />
+      <mass value="5.0"/>
+      <origin xyz="0.25 0 0" rpy="0 0 0"/>
+      <inertia ixx="0.1" ixy="0" ixz="0" iyy="0.5" iyz="0" izz="0.5" />
     </inertial>
-    <visual><origin xyz="0.15 0.0 0.0" rpy="0 0 0"/><geometry><box size="1.02 0.12 0.12"/></geometry></visual>
-    <visual><origin xyz="0.6 0.0 -0.15" rpy="0 0 0"/><geometry><box size="0.12 0.12 0.3"/></geometry></visual>
-    <visual><origin xyz="-0.3 0.0 -0.075" rpy="0 0 0"/><geometry><box size="0.12 0.12 0.15"/></geometry></visual>
-    <collision><origin xyz="0.15 0.0 -0.075" rpy="0 0 0"/><geometry><box size="0.9 0.06 0.15"/></geometry></collision>
+    <visual><origin xyz="0.25 0 0"/><geometry><box size="1.7 0.2 0.2"/></geometry></visual>
   </link>
   <gazebo reference="left_rocker_arm"><material>Gazebo/DarkGrey</material></gazebo>
   <joint name="left_differential_axle" type="revolute">
-    <origin xyz="0.0 0.39 0.0" rpy="0 0 0"/>
+    <origin xyz="0.0 0.65 0" rpy="0 0 0"/>
     <parent link="base_link"/>
     <child link="left_rocker_arm"/>
-    <axis xyz="0.0 3.0 0.0"/>
-    <!-- ADVANCED MECHANICS: Mechanical Hard Stops.
-         Changed from continuous back to revolute, but with strictly tuned limits
-         (+/- 0.6 radians). This simulates the physical chassis bumping against
-         the arm, preventing the robot from doing a full backflip over its own wheels. -->
-    <limit lower="-0.6" upper="0.6" effort="1000" velocity="10"/>
-    <dynamics damping="8.0" friction="2.0"/>
+    <axis xyz="0 1 0"/>
+    <limit lower="-0.6" upper="0.6" effort="10000" velocity="5"/>
+    <dynamics damping="100.0" friction="50.0"/>
   </joint>
-  <!-- Instantiate Left Front Wheel -->
-  <xacro:boc_wheel name="front_left_wheel" parent="left_rocker_arm" origin_xyz="1.8 0.54 -0.9"/>
+  <!-- Front Left Wheel: X=1.0, Y=0.2, Z=-0.5 -->
+  <xacro:boc_wheel name="front_left_wheel" parent="left_rocker_arm" origin_xyz="1.0 0.2 -0.5"/>
   <link name="left_bogie_link">
     <inertial>
-      <mass value="0.5"/>
-      <origin xyz="0.0 0.0 0.0" rpy="0 0 0"/>
-      <inertia ixx="0.005" ixy="0" ixz="0" iyy="0.005" iyz="0" izz="0.005" />
+      <mass value="4.0"/>
+      <origin xyz="0 0 0" rpy="0 0 0"/>
+      <inertia ixx="0.1" ixy="0" ixz="0" iyy="0.3" iyz="0" izz="0.3" />
     </inertial>
-    <visual><origin xyz="0.0 0.0 0.0" rpy="0 0 0"/><geometry><box size="0.72 0.12 0.12"/></geometry></visual>
-    <visual><origin xyz="0.3 0.0 -0.075" rpy="0 0 0"/><geometry><box size="0.12 0.12 0.15"/></geometry></visual>
-    <visual><origin xyz="-0.3 0.0 -0.075" rpy="0 0 0"/><geometry><box size="0.12 0.12 0.15"/></geometry></visual>
-    <collision><origin xyz="0.0 0.0 -0.075" rpy="0 0 0"/><geometry><box size="0.6 0.06 0.15"/></geometry></collision>
+    <visual><origin xyz="0 0 0"/><geometry><box size="1.2 0.2 0.2"/></geometry></visual>
   </link>
   <gazebo reference="left_bogie_link"><material>Gazebo/DarkGrey</material></gazebo>
   <joint name="left_bogie_pivot" type="revolute">
-    <origin xyz="-0.3 0.0 -0.15" rpy="0 0 0"/>
+    <origin xyz="-0.5 0 -0.2" rpy="0 0 0"/>
     <parent link="left_rocker_arm"/>
     <child link="left_bogie_link"/>
-    <axis xyz="0.0 3.0 0.0"/>
-    <!-- Mechanical stop for the bogie (+/- 0.8 radians) -->
-    <limit lower="-0.8" upper="0.8" effort="500" velocity="10"/>
-    <dynamics damping="3.0" friction="1.0"/>
+    <axis xyz="0 1 0"/>
+    <limit lower="-0.8" upper="0.8" effort="5000" velocity="5"/>
+    <dynamics damping="50.0" friction="20.0"/>
   </joint>
-  <!-- Instantiate Left Mid & Rear Wheels -->
-  <xacro:boc_wheel name="mid_left_wheel" parent="left_bogie_link" origin_xyz="0.9 0.54 -0.45"/>
-  <xacro:boc_wheel name="back_left_wheel" parent="left_bogie_link" origin_xyz="-0.9 0.54 -0.45"/>
+  <xacro:boc_wheel name="mid_left_wheel" parent="left_bogie_link" origin_xyz="0.5 0.2 -0.3"/>
+  <xacro:boc_wheel name="back_left_wheel" parent="left_bogie_link" origin_xyz="-0.5 0.2 -0.3"/>
   <!-- =============================== -->
   <!-- RIGHT SIDE ASSEMBLY             -->
@@ -171,46 +127,39 @@
   <link name="right_rocker_arm">
     <inertial>
-      <mass value="0.5"/>
-      <origin xyz="0.15 0.0 0.0" rpy="0 0 0"/>
-      <inertia ixx="0.005" ixy="0" ixz="0" iyy="0.005" iyz="0" izz="0.005" />
+      <mass value="5.0"/>
+      <origin xyz="0.25 0 0" rpy="0 0 0"/>
+      <inertia ixx="0.1" ixy="0" ixz="0" iyy="0.5" iyz="0" izz="0.5" />
     </inertial>
-    <visual><origin xyz="0.15 0.0 0.0" rpy="0 0 0"/><geometry><box size="1.02 0.12 0.12"/></geometry></visual>
-    <visual><origin xyz="0.6 0.0 -0.15" rpy="0 0 0"/><geometry><box size="0.12 0.12 0.3"/></geometry></visual>
-    <visual><origin xyz="-0.3 0.0 -0.075" rpy="0 0 0"/><geometry><box size="0.12 0.12 0.15"/></geometry></visual>
-    <collision><origin xyz="0.15 0.0 -0.075" rpy="0 0 0"/><geometry><box size="0.9 0.06 0.15"/></geometry></collision>
+    <visual><origin xyz="0.25 0 0"/><geometry><box size="1.7 0.2 0.2"/></geometry></visual>
   </link>
   <gazebo reference="right_rocker_arm"><material>Gazebo/DarkGrey</material></gazebo>
   <joint name="right_differential_axle" type="revolute">
-    <origin xyz="0.0 -0.39 0.0" rpy="0 0 0"/>
+    <origin xyz="0.0 -0.65 0" rpy="0 0 0"/>
     <parent link="base_link"/>
     <child link="right_rocker_arm"/>
-    <axis xyz="0.0 3.0 0.0"/>
-    <limit lower="-0.6" upper="0.6" effort="1000" velocity="10"/>
-    <dynamics damping="8.0" friction="2.0"/>
+    <axis xyz="0 1 0"/>
+    <limit lower="-0.6" upper="0.6" effort="10000" velocity="5"/>
+    <dynamics damping="100.0" friction="50.0"/>
   </joint>
-  <!-- Instantiate Right Front Wheel -->
-  <xacro:boc_wheel name="front_right_wheel" parent="right_rocker_arm" origin_xyz="1.8 -0.54 -0.9"/>
+  <!-- Front Right Wheel -->
+  <xacro:boc_wheel name="front_right_wheel" parent="right_rocker_arm" origin_xyz="1.0 -0.2 -0.5"/>
   <link name="right_bogie_link">
     <inertial>
-      <mass value="0.5"/>
-      <origin xyz="0.0 0.0 0.0" rpy="0 0 0"/>
-      <inertia ixx="0.005" ixy="0" ixz="0" iyy="0.005" iyz="0" izz="0.005" />
+      <mass value="4.0"/>
+      <origin xyz="0 0 0" rpy="0 0 0"/>
+      <inertia ixx="0.1" ixy="0" ixz="0" iyy="0.3" iyz="0" izz="0.3" />
     </inertial>
-    <visual><origin xyz="0.0 0.0 0.0" rpy="0 0 0"/><geometry><box size="0.72 0.12 0.12"/></geometry></visual>
-    <visual><origin xyz="0.3 0.0 -0.075" rpy="0 0 0"/><geometry><box size="0.12 0.12 0.15"/></geometry></visual>
-    <visual><origin xyz="-0.3 0.0 -0.075" rpy="0 0 0"/><geometry><box size="0.12 0.12 0.15"/></geometry></visual>
-    <collision><origin xyz="0.0 0.0 -0.075" rpy="0 0 0"/><geometry><box size="0.6 0.06 0.15"/></geometry></collision>
+    <visual><origin xyz="0 0 0"/><geometry><box size="1.2 0.2 0.2"/></geometry></visual>
   </link>
   <gazebo reference="right_bogie_link"><material>Gazebo/DarkGrey</material></gazebo>
   <joint name="right_bogie_pivot" type="revolute">
-    <origin xyz="-0.3 0.0 -0.15" rpy="0 0 0"/>
+    <origin xyz="-0.5 0 -0.2" rpy="0 0 0"/>
     <parent link="right_rocker_arm"/>
     <child link="right_bogie_link"/>
-    <axis xyz="0.0 3.0 0.0"/>
-    <limit lower="-0.8" upper="0.8" effort="500" velocity="10"/>
-    <dynamics damping="3.0" friction="1.0"/>
+    <axis xyz="0 1 0"/>
+    <limit lower="-0.8" upper="0.8" effort="5000" velocity="5"/>
+    <dynamics damping="50.0" friction="20.0"/>
   </joint>
-  <!-- Instantiate Right Mid & Rear Wheels -->
-  <xacro:boc_wheel name="mid_right_wheel" parent="right_bogie_link" origin_xyz="0.9 -0.54 -0.45"/>
-  <xacro:boc_wheel name="back_right_wheel" parent="right_bogie_link" origin_xyz="-0.9 -0.54 -0.45"/>
+  <xacro:boc_wheel name="mid_right_wheel" parent="right_bogie_link" origin_xyz="0.5 -0.2 -0.3"/>
+  <xacro:boc_wheel name="back_right_wheel" parent="right_bogie_link" origin_xyz="-0.5 -0.2 -0.3"/>
 </robot>
